File: sch/sch.sch (KiCad schematic (older format))
At the start: 16 parts

Commit message: pcb
Parts:
- removed J?: USB_A, symbol Connector:USB_A
- added J1: swd, local:3WIRE_PADS, symbol Connector:Conn_01x03
- added J3: USB, local:4_wire, symbol Connector:Conn_01x04
- added R1, R2: 50, Resistor_SMD:R_0402_1005Metric, symbol device:R
- added R4: 10, Resistor_SMD:R_0805_2012Metric, symbol device:R
- C1, C2, C3, C4, C5, C6, C7, C8, C9: renamed from C?; footprint (none) -> Capacitor_SMD:C_0805_2012Metric
- C10: renamed from C?; value 0.1uF -> 10uF; footprint (none) -> Capacitor_SMD:C_0805_2012Metric
- J2: renamed from J?; footprint (none) -> local:8Bit_wire
- R3: renamed from R?; footprint (none) -> Resistor_SMD:R_0402_1005Metric
- U1: renamed from U?; footprint Housings_QFP:LQFP-48_7x7mm_Pitch0.5mm -> Package_QFP:LQFP-48_7x7mm_P0.5mm
- U2: renamed from U?; footprint TO_SOT_Packages_SMD:SOT-89-3 -> Package_TO_SOT_SMD:SOT-89-3
- Y1: renamed from Y?; footprint (none) -> Crystal:Crystal_SMD_5032-2Pin_5.0x3.2mm
Connections:
- net labels added: SWCLK, SWDIO
- wire segments 85 -> 96
- no-connect marks 25 -> 20
Other:
- moved on the sheet: C10, C4, C5, C6, C7, C8, C9, J2, R3

Commit message: sch corrections
Connections:
- wire segments 96 -> 95
- no-connect marks 20 -> 22
Changed lines of the file:
@@
 Wire Wire Line
 	7700 5550 7750 5550
-Wire Wire Line
-	6200 5000 6450 5000
-Entry Wire Line
-	6450 5000 6550 5100
 $Comp
 L local:STM32F103C8Tx_usb U1
@@
 Wire Wire Line
 	4950 5000 5100 5000
+NoConn ~ 5100 4900
+NoConn ~ 6200 5000
 Wire Bus Line
 	4850 5750 7050 5750

Commit message: buttons
Parts:
- added J4: JOYSTICK, symbol Connector:Conn_01x07
- added SW1: SW_LEFT, symbol Switch:SW_Push
- added SW2: SW_UP, symbol Switch:SW_Push
- added SW3: SW_RIGHT, symbol Switch:SW_Push
- added SW4: SW_DOWN, symbol Switch:SW_Push
- added SW5: SW_1, symbol Switch:SW_Push
- added SW6: SW_2, symbol Switch:SW_Push
Connections:
- wire segments 95 -> 126
Other:
- moved on the sheet: C1, C10, C2, C3, C4, C5, C6, C7, C8, C9, J1, J2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

Commit message: err in pcb
Parts:
- removed U2: L78L33_SOT89, Package_TO_SOT_SMD:SOT-89-3, symbol regul:L78L33_SOT89
- added U2: XC6206-33, Package_TO_SOT_SMD:SOT-23, symbol local:XC6206-33
Changed lines of the file:
@@
 L power:+5V #PWR0101
 U 1 1 60BA6D79
-P 7050 3300
-F 0 "#PWR0101" H 7050 3150 50  0001 C CNN
-F 1 "+5V" H 7100 3450 50  0000 C CNN
-F 2 "" H 7050 3300 50  0001 C CNN
-F 3 "" H 7050 3300 50  0001 C CNN
-	1    7050 3300
-	1    0    0    -1
-$EndComp
-$Comp
-L power:+3.3V #PWR0102
-U 1 1 60BAE187
-P 6950 3300
-F 0 "#PWR0102" H 6950 3150 50  0001 C CNN
-F 1 "+3.3V" H 6900 3450 50  0000 C CNN
-F 2 "" H 6950 3300 50  0001 C CNN
-F 3 "" H 6950 3300 50  0001 C CNN
-	1    6950 3300
-	1    0    0    -1
-$EndComp
-Wire Wire Line
-	6950 3350 6950 3300
+P 7050 3250
+F 0 "#PWR0101" H 7050 3100 50  0001 C CNN
+F 1 "+5V" H 7100 3400 50  0000 C CNN
+F 2 "" H 7050 3250 50  0001 C CNN
+F 3 "" H 7050 3250 50  0001 C CNN
+	1    7050 3250
+	1    0    0    -1
+$EndComp
 $Comp
 L device:Crystal Y1
@@
 	1    0    0    -1
 $EndComp
-$Comp
-L regul:L78L33_SOT89 U2
-U 1 1 60B98975
-P 6050 1750
-F 0 "U2" H 6400 1900 50  0000 C CNN
-F 1 "L78L33_SOT89" H 6050 1901 50  0000 C CNN
-F 2 "Package_TO_SOT_SMD:SOT-89-3" H 6050 1950 50  0001 C CIN
-F 3 "http://www.st.com/content/ccc/resource/technical/document/datasheet/15/55/e5/aa/23/5b/43/fd/CD00000446.pdf/files/CD00000446.pdf/jcr:content/translations/en.CD00000446.pdf" H 6050 1700 50  0001 C CNN
-	1    6050 1750
-	1    0    0    -1
-$EndComp
 Entry Bus Bus
 	6300 5650 6400 5750
@@
 	7050 3600 7100 3600
 Wire Wire Line
-	7050 3300 7050 3600
-Wire Wire Line
 	7050 3950 7050 3900
 Wire Wire Line
@@
 Wire Wire Line
 	8550 5550 8800 5550
+$Comp
+L local:XC6206-33 U2
+U 1 1 61038F36
+P 6050 1750
+F 0 "U2" H 6050 1992 50  0000 C CNN
+F 1 "XC6206-33" H 6050 1901 50  0000 C CNN
+F 2 "Package_TO_SOT_SMD:SOT-23" H 6050 1750 50  0001 C CNN
+F 3 "" H 6150 1500 50  0001 C CNN
+	1    6050 1750
+	1    0    0    -1
+$EndComp
+Wire Wire Line
+	7050 3250 7050 3600
+$Comp
+L power:+3.3V #PWR0102
+U 1 1 6105D4FC
+P 6950 3250
+F 0 "#PWR0102" H 6950 3100 50  0001 C CNN
+F 1 "+3.3V" H 6900 3400 50  0000 C CNN
+F 2 "" H 6950 3250 50  0001 C CNN
+F 3 "" H 6950 3250 50  0001 C CNN
+	1    6950 3250
+	1    0    0    -1
+$EndComp
+Wire Wire Line
+	6950 3350 6950 3250
 Wire Bus Line
 	4200 5750 6400 5750

Commit message: begin to write normal documentation
Parts:
- R3: value 100k -> 4.7k
Changed lines of the file:
@@
 P 6950 3500
 F 0 "R3" H 6800 3550 50  0000 L CNN
-F 1 "100k" V 6950 3400 50  0000 L CNN
+F 1 "4.7k" V 6950 3400 50  0000 L CNN
 F 2 "Resistor_SMD:R_0402_1005Metric" V 6880 3500 50  0001 C CNN
 F 3 "" H 6950 3500 50  0001 C CNN

Commit message: *
Parts:
- C1, C10, C2, C3, C4, C5, C6, C7, C8, C9: symbol device:C -> sch-rescue:C-device
- J1: symbol Connector:Conn_01x03 -> sch-rescue:Conn_01x03-Connector
- J2: symbol Connector:Conn_01x09 -> sch-rescue:Conn_01x09-Connector
- J3: symbol Connector:Conn_01x04 -> sch-rescue:Conn_01x04-Connector
- J4: symbol Connector:Conn_01x07 -> sch-rescue:Conn_01x07-Connector
- R1, R2, R3, R4: symbol device:R -> sch-rescue:R-device
- SW1, SW2, SW3, SW4, SW5, SW6: symbol Switch:SW_Push -> sch-rescue:SW_Push-Switch
- Y1: symbol device:Crystal -> sch-rescue:Crystal-device
Changed lines of the file:
@@
 $EndDescr
 $Comp
-L device:R R3
+L sch-rescue:R-device R3
 U 1 1 60B98022
 P 6950 3500
@@
 $EndComp
 $Comp
-L power:+5V #PWR0101
+L sch-rescue:+5V-power #PWR0101
 U 1 1 60BA6D79
 P 7050 3250
@@
 $EndComp
 $Comp
-L device:Crystal Y1
+L sch-rescue:Crystal-device Y1
 U 1 1 60BB7B29
 P 4200 2850
@@
 $EndComp
 $Comp
-L device:C C1
+L sch-rescue:C-device C1
 U 1 1 60BBCAE9
 P 3900 2700
@@
 $EndComp
 $Comp
-L device:C C2
+L sch-rescue:C-device C2
 U 1 1 60BBD52B
 P 3900 3000
@@
 Connection ~ 4200 3000
 $Comp
-L power:GND #PWR0103
+L sch-rescue:GND-power #PWR0103
 U 1 1 60BC5327
 P 3650 3050
@@
 Connection ~ 3650 3000
 $Comp
-L device:C C5
+L sch-rescue:C-device C5
 U 1 1 60BCC99C
 P 5800 2850
@@
 $EndComp
 $Comp
-L power:GND #PWR0104
+L sch-rescue:GND-power #PWR0104
 U 1 1 60BCEBAF
 P 5800 3050
@@
 $EndComp
 $Comp
-L power:+3.3V #PWR0105
+L sch-rescue:+3.3V-power #PWR0105
 U 1 1 60BCF857
 P 5800 2650
@@
 $EndComp
 $Comp
-L device:C C6
+L sch-rescue:C-device C6
 U 1 1 60BD3987
 P 6050 2850
@@
 $EndComp
 $Comp
-L power:GND #PWR0106
+L sch-rescue:GND-power #PWR0106
 U 1 1 60BD398D
 P 6050 3050
@@
 $EndComp
 $Comp
-L power:+3.3V #PWR0107
+L sch-rescue:+3.3V-power #PWR0107
 U 1 1 60BD3993
 P 6050 2650
@@
 $EndComp
 $Comp
-L device:C C7
+L sch-rescue:C-device C7
 U 1 1 60BD4708
 P 6300 2850
@@
 $EndComp
 $Comp
-L power:GND #PWR0108
+L sch-rescue:GND-power #PWR0108
 U 1 1 60BD470E
 P 6300 3050
@@
 $EndComp
 $Comp
-L power:+3.3V #PWR0109
+L sch-rescue:+3.3V-power #PWR0109
 U 1 1 60BD4714
 P 6300 2650
@@
 $EndComp
 $Comp
-L device:C C9
+L sch-rescue:C-device C9
 U 1 1 60BD5497
 P 6550 2850
@@
 $EndComp
 $Comp
-L power:GND #PWR0110
+L sch-rescue:GND-power #PWR0110
 U 1 1 60BD549D
 P 6550 3050
@@
 $EndComp
 $Comp
-L power:+3.3V #PWR0111
+L sch-rescue:+3.3V-power #PWR0111
 U 1 1 60BD54A3
 P 6550 2650
@@
 	6300 2650 6300 2700
 $Comp
-L power:+3.3V #PWR0112
+L sch-rescue:+3.3V-power #PWR0112
 U 1 1 60BE41C5
 P 5100 1700
@@
 Connection ~ 5100 1750
 $Comp
-L power:GND #PWR0113
+L sch-rescue:GND-power #PWR0113
 U 1 1 60BE8B74
 P 5100 5500
@@
 	4900 5450 5000 5450
 $Comp
-L power:GND #PWR0114
+L sch-rescue:GND-power #PWR0114
 U 1 1 60BFBFA2
 P 7050 3950
@@
 $EndComp
 $Comp
-L power:GND #PWR0115
+L sch-rescue:GND-power #PWR0115
 U 1 1 60C02E98
 P 4000 2400
@@
 $EndComp
 $Comp
-L device:C C3
+L sch-rescue:C-device C3
 U 1 1 60C06DEC
 P 4200 2200
@@
 $EndComp
 $Comp
-L power:GND #PWR0116
+L sch-rescue:GND-power #PWR0116
 U 1 1 60C0A725
 P 4000 2200
@@
 	4000 2400 4450 2400
 $Comp
-L power:+3.3V #PWR0117
+L sch-rescue:+3.3V-power #PWR0117
 U 1 1 60C17286
 P 4400 2550
@@
 	5900 5650 6000 5750
 $Comp
-L Connector:Conn_01x09 J2
+L sch-rescue:Conn_01x09-Connector J2
 U 1 1 60C72175
 P 7300 5150
@@
 JOY7
 $Comp
-L power:GND #PWR0118
+L sch-rescue:GND-power #PWR0118
 U 1 1 60CB8790
 P 7050 5600
@@
 	5700 1750 5700 1700
 $Comp
-L power:+3.3V #PWR0119
+L sch-rescue:+3.3V-power #PWR0119
 U 1 1 60BDEA7C
 P 5700 1700
@@
 $EndComp
 $Comp
-L power:+5V #PWR0120
+L sch-rescue:+5V-power #PWR0120
 U 1 1 60BDCB44
 P 7150 1700
@@
 	5700 2050 5700 2100
 $Comp
-L power:GND #PWR0121
+L sch-rescue:GND-power #PWR0121
 U 1 1 60BA3E87
 P 6650 2150
@@
 	5750 1750 5700 1750
 $Comp
-L device:C C8
+L sch-rescue:C-device C8
 U 1 1 60B9D265
 P 6400 1900
@@
 $EndComp
 $Comp
-L device:C C10
+L sch-rescue:C-device C10
 U 1 1 60B9CD1A
 P 6650 1900
@@
 $EndComp
 $Comp
-L device:C C4
+L sch-rescue:C-device C4
 U 1 1 60B9CA4E
 P 5700 1900
@@
 	6300 5650 6400 5750
 $Comp
-L device:R R2
+L sch-rescue:R-device R2
 U 1 1 60BAF8CE
 P 6700 3800
@@
 $EndComp
 $Comp
-L Connector:Conn_01x03 J1
+L sch-rescue:Conn_01x03-Connector J1
 U 1 1 60BDE5E6
 P 7300 4300
@@
 	6300 4500 6400 4400
 $Comp
-L power:GND #PWR0122
+L sch-rescue:GND-power #PWR0122
 U 1 1 60BEBAA9
 P 7050 4450
@@
 	5800 4800 5550 4800
 $Comp
-L device:R R4
+L sch-rescue:R-device R4
 U 1 1 60BAA748
 P 6950 1750
@@
 	7100 1750 7150 1750
 $Comp
-L Connector:Conn_01x04 J3
+L sch-rescue:Conn_01x04-Connector J3
 U 1 1 60BD2978
 P 7300 3700
@@
 	6300 3800 6400 3700
 $Comp
-L device:R R1
+L sch-rescue:R-device R1
 U 1 1 60BAF3EA
 P 6700 3700
@@
 NoConn ~ 4450 3300
 $Comp
-L power:GND #PWR0123
+L sch-rescue:GND-power #PWR0123
 U 1 1 60D66AD7
 P 4300 5050
@@
 NoConn ~ 5550 5000
 $Comp
-L Connector:Conn_01x07 J4
+L sch-rescue:Conn_01x07-Connector J4
 U 1 1 60E21F7B
 P 8200 5250
@@
 $EndComp
 $Comp
-L Switch:SW_Push SW6
+L sch-rescue:SW_Push-Switch SW6
 U 1 1 60E2AE97
 P 9000 5700
@@
 $EndComp
 $Comp
-L Switch:SW_Push SW5
+L sch-rescue:SW_Push-Switch SW5
 U 1 1 60E2BB79
 P 9000 5550
@@
 $EndComp
 $Comp
-L Switch:SW_Push SW4
+L sch-rescue:SW_Push-Switch SW4
 U 1 1 60E2DB4C
 P 9000 5400
@@
 $EndComp
 $Comp
-L Switch:SW_Push SW3
+L sch-rescue:SW_Push-Switch SW3
 U 1 1 60E2DDFE
 P 9000 5250
@@
 $EndComp
 $Comp
-L Switch:SW_Push SW2
+L sch-rescue:SW_Push-Switch SW2
 U 1 1 60E2E03E
 P 9000 5100
@@
 $EndComp
 $Comp
-L Switch:SW_Push SW1
+L sch-rescue:SW_Push-Switch SW1
 U 1 1 60E2E395
 P 9000 4950
@@
 	7050 3250 7050 3600
 $Comp
-L power:+3.3V #PWR0102
+L sch-rescue:+3.3V-power #PWR0102
 U 1 1 6105D4FC
 P 6950 3250

Commit message: убрался в файлах
Parts:
- C1, C10, C2, C3, C4, C5, C6, C7, C8, C9: symbol sch-rescue:C-device -> sch-rescue:C-device-sch-rescue
- J1: symbol sch-rescue:Conn_01x03-Connector -> sch-rescue:Conn_01x03-Connector-sch-rescue
- J2: symbol sch-rescue:Conn_01x09-Connector -> sch-rescue:Conn_01x09-Connector-sch-rescue
- J3: symbol sch-rescue:Conn_01x04-Connector -> sch-rescue:Conn_01x04-Connector-sch-rescue
- J4: symbol sch-rescue:Conn_01x07-Connector -> sch-rescue:Conn_01x07-Connector-sch-rescue
- R1, R2, R3, R4: symbol sch-rescue:R-device -> sch-rescue:R-device-sch-rescue
- SW1, SW2, SW3, SW4, SW5, SW6: symbol sch-rescue:SW_Push-Switch -> sch-rescue:SW_Push-Switch-sch-rescue
- Y1: symbol sch-rescue:Crystal-device -> sch-rescue:Crystal-device-sch-rescue
Changed lines of the file:
@@
 $EndDescr
 $Comp
-L sch-rescue:R-device R3
+L sch-rescue:R-device-sch-rescue R3
 U 1 1 60B98022
 P 6950 3500
@@
 $EndComp
 $Comp
-L sch-rescue:+5V-power #PWR0101
+L sch-rescue:+5V-power-sch-rescue #PWR0101
 U 1 1 60BA6D79
 P 7050 3250
@@
 $EndComp
 $Comp
-L sch-rescue:Crystal-device Y1
+L sch-rescue:Crystal-device-sch-rescue Y1
 U 1 1 60BB7B29
 P 4200 2850
@@
 $EndComp
 $Comp
-L sch-rescue:C-device C1
+L sch-rescue:C-device-sch-rescue C1
 U 1 1 60BBCAE9
 P 3900 2700
@@
 $EndComp
 $Comp
-L sch-rescue:C-device C2
+L sch-rescue:C-device-sch-rescue C2
 U 1 1 60BBD52B
 P 3900 3000
@@
 Connection ~ 4200 3000
 $Comp
-L sch-rescue:GND-power #PWR0103
+L sch-rescue:GND-power-sch-rescue #PWR0103
 U 1 1 60BC5327
 P 3650 3050
@@
 Connection ~ 3650 3000
 $Comp
-L sch-rescue:C-device C5
+L sch-rescue:C-device-sch-rescue C5
 U 1 1 60BCC99C
 P 5800 2850
@@
 $EndComp
 $Comp
-L sch-rescue:GND-power #PWR0104
+L sch-rescue:GND-power-sch-rescue #PWR0104
 U 1 1 60BCEBAF
 P 5800 3050
@@
 $EndComp
 $Comp
-L sch-rescue:+3.3V-power #PWR0105
+L sch-rescue:+3.3V-power-sch-rescue #PWR0105
 U 1 1 60BCF857
 P 5800 2650
@@
 $EndComp
 $Comp
-L sch-rescue:C-device C6
+L sch-rescue:C-device-sch-rescue C6
 U 1 1 60BD3987
 P 6050 2850
@@
 $EndComp
 $Comp
-L sch-rescue:GND-power #PWR0106
+L sch-rescue:GND-power-sch-rescue #PWR0106
 U 1 1 60BD398D
 P 6050 3050
@@
 $EndComp
 $Comp
-L sch-rescue:+3.3V-power #PWR0107
+L sch-rescue:+3.3V-power-sch-rescue #PWR0107
 U 1 1 60BD3993
 P 6050 2650
@@
 $EndComp
 $Comp
-L sch-rescue:C-device C7
+L sch-rescue:C-device-sch-rescue C7
 U 1 1 60BD4708
 P 6300 2850
@@
 $EndComp
 $Comp
-L sch-rescue:GND-power #PWR0108
+L sch-rescue:GND-power-sch-rescue #PWR0108
 U 1 1 60BD470E
 P 6300 3050
@@
 $EndComp
 $Comp
-L sch-rescue:+3.3V-power #PWR0109
+L sch-rescue:+3.3V-power-sch-rescue #PWR0109
 U 1 1 60BD4714
 P 6300 2650
@@
 $EndComp
 $Comp
-L sch-rescue:C-device C9
+L sch-rescue:C-device-sch-rescue C9
 U 1 1 60BD5497
 P 6550 2850
@@
 $EndComp
 $Comp
-L sch-rescue:GND-power #PWR0110
+L sch-rescue:GND-power-sch-rescue #PWR0110
 U 1 1 60BD549D
 P 6550 3050
@@
 $EndComp
 $Comp
-L sch-rescue:+3.3V-power #PWR0111
+L sch-rescue:+3.3V-power-sch-rescue #PWR0111
 U 1 1 60BD54A3
 P 6550 2650
@@
 	6300 2650 6300 2700
 $Comp
-L sch-rescue:+3.3V-power #PWR0112
+L sch-rescue:+3.3V-power-sch-rescue #PWR0112
 U 1 1 60BE41C5
 P 5100 1700
@@
 Connection ~ 5100 1750
 $Comp
-L sch-rescue:GND-power #PWR0113
+L sch-rescue:GND-power-sch-rescue #PWR0113
 U 1 1 60BE8B74
 P 5100 5500
@@
 	4900 5450 5000 5450
 $Comp
-L sch-rescue:GND-power #PWR0114
+L sch-rescue:GND-power-sch-rescue #PWR0114
 U 1 1 60BFBFA2
 P 7050 3950
@@
 $EndComp
 $Comp
-L sch-rescue:GND-power #PWR0115
+L sch-rescue:GND-power-sch-rescue #PWR0115
 U 1 1 60C02E98
 P 4000 2400
@@
 $EndComp
 $Comp
-L sch-rescue:C-device C3
+L sch-rescue:C-device-sch-rescue C3
 U 1 1 60C06DEC
 P 4200 2200
@@
 $EndComp
 $Comp
-L sch-rescue:GND-power #PWR0116
+L sch-rescue:GND-power-sch-rescue #PWR0116
 U 1 1 60C0A725
 P 4000 2200
@@
 	4000 2400 4450 2400
 $Comp
-L sch-rescue:+3.3V-power #PWR0117
+L sch-rescue:+3.3V-power-sch-rescue #PWR0117
 U 1 1 60C17286
 P 4400 2550
@@
 	5900 5650 6000 5750
 $Comp
-L sch-rescue:Conn_01x09-Connector J2
+L sch-rescue:Conn_01x09-Connector-sch-rescue J2
 U 1 1 60C72175
 P 7300 5150
@@
 JOY7
 $Comp
-L sch-rescue:GND-power #PWR0118
+L sch-rescue:GND-power-sch-rescue #PWR0118
 U 1 1 60CB8790
 P 7050 5600
@@
 	5700 1750 5700 1700
 $Comp
-L sch-rescue:+3.3V-power #PWR0119
+L sch-rescue:+3.3V-power-sch-rescue #PWR0119
 U 1 1 60BDEA7C
 P 5700 1700
@@
 $EndComp
 $Comp
-L sch-rescue:+5V-power #PWR0120
+L sch-rescue:+5V-power-sch-rescue #PWR0120
 U 1 1 60BDCB44
 P 7150 1700
@@
 	5700 2050 5700 2100
 $Comp
-L sch-rescue:GND-power #PWR0121
+L sch-rescue:GND-power-sch-rescue #PWR0121
 U 1 1 60BA3E87
 P 6650 2150
@@
 	5750 1750 5700 1750
 $Comp
-L sch-rescue:C-device C8
+L sch-rescue:C-device-sch-rescue C8
 U 1 1 60B9D265
 P 6400 1900
@@
 $EndComp
 $Comp
-L sch-rescue:C-device C10
+L sch-rescue:C-device-sch-rescue C10
 U 1 1 60B9CD1A
 P 6650 1900
@@
 $EndComp
 $Comp
-L sch-rescue:C-device C4
+L sch-rescue:C-device-sch-rescue C4
 U 1 1 60B9CA4E
 P 5700 1900
@@
 	6300 5650 6400 5750
 $Comp
-L sch-rescue:R-device R2
+L sch-rescue:R-device-sch-rescue R2
 U 1 1 60BAF8CE
 P 6700 3800
@@
 $EndComp
 $Comp
-L sch-rescue:Conn_01x03-Connector J1
+L sch-rescue:Conn_01x03-Connector-sch-rescue J1
 U 1 1 60BDE5E6
 P 7300 4300
@@
 	6300 4500 6400 4400
 $Comp
-L sch-rescue:GND-power #PWR0122
+L sch-rescue:GND-power-sch-rescue #PWR0122
 U 1 1 60BEBAA9
 P 7050 4450
@@
 	5800 4800 5550 4800
 $Comp
-L sch-rescue:R-device R4
+L sch-rescue:R-device-sch-rescue R4
 U 1 1 60BAA748
 P 6950 1750
@@
 	7100 1750 7150 1750
 $Comp
-L sch-rescue:Conn_01x04-Connector J3
+L sch-rescue:Conn_01x04-Connector-sch-rescue J3
 U 1 1 60BD2978
 P 7300 3700
@@
 	6300 3800 6400 3700
 $Comp
-L sch-rescue:R-device R1
+L sch-rescue:R-device-sch-rescue R1
 U 1 1 60BAF3EA
 P 6700 3700
@@
 NoConn ~ 4450 3300
 $Comp
-L sch-rescue:GND-power #PWR0123
+L sch-rescue:GND-power-sch-rescue #PWR0123
 U 1 1 60D66AD7
 P 4300 5050
@@
 NoConn ~ 5550 5000
 $Comp
-L sch-rescue:Conn_01x07-Connector J4
+L sch-rescue:Conn_01x07-Connector-sch-rescue J4
 U 1 1 60E21F7B
 P 8200 5250
@@
 $EndComp
 $Comp
-L sch-rescue:SW_Push-Switch SW6
+L sch-rescue:SW_Push-Switch-sch-rescue SW6
 U 1 1 60E2AE97
 P 9000 5700
@@
 $EndComp
 $Comp
-L sch-rescue:SW_Push-Switch SW5
+L sch-rescue:SW_Push-Switch-sch-rescue SW5
 U 1 1 60E2BB79
 P 9000 5550
@@
 $EndComp
 $Comp
-L sch-rescue:SW_Push-Switch SW4
+L sch-rescue:SW_Push-Switch-sch-rescue SW4
 U 1 1 60E2DB4C
 P 9000 5400
@@
 $EndComp
 $Comp
-L sch-rescue:SW_Push-Switch SW3
+L sch-rescue:SW_Push-Switch-sch-rescue SW3
 U 1 1 60E2DDFE
 P 9000 5250
@@
 $EndComp
 $Comp
-L sch-rescue:SW_Push-Switch SW2
+L sch-rescue:SW_Push-Switch-sch-rescue SW2
 U 1 1 60E2E03E
 P 9000 5100
@@
 $EndComp
 $Comp
-L sch-rescue:SW_Push-Switch SW1
+L sch-rescue:SW_Push-Switch-sch-rescue SW1
 U 1 1 60E2E395
 P 9000 4950
@@
 	7050 3250 7050 3600
 $Comp
-L sch-rescue:+3.3V-power #PWR0102
+L sch-rescue:+3.3V-power-sch-rescue #PWR0102
 U 1 1 6105D4FC
 P 6950 3250
