File: sch/remote/remote.sch (KiCad schematic (older format))
At the start: 24 parts, among them J1 swd, J2 power_sw, J3 USB_A, Q1 DTD114E, U1 STM32F103C8Tx_usb, U2 XC6206-33, U3 TSOP17xx, Y1 8M

Commit message: 0402 caps
Parts:
- C1, C2, C3, C5, C6, C7, C8, C9: footprint Capacitor_SMD:C_0805_2012Metric -> Capacitor_SMD:C_0402_1005Metric
Changed lines of the file:
@@
 F 0 "C1" H 3900 2800 50  0000 L CNN
 F 1 "22p" H 3900 2600 50  0000 L CNN
-F 2 "Capacitor_SMD:C_0805_2012Metric" H 3938 2550 50  0001 C CNN
+F 2 "Capacitor_SMD:C_0402_1005Metric" H 3938 2550 50  0001 C CNN
 F 3 "" H 3900 2700 50  0001 C CNN
 	1    3900 2700
@@
 F 0 "C2" H 3900 3100 50  0000 L CNN
 F 1 "22p" H 3900 2900 50  0000 L CNN
-F 2 "Capacitor_SMD:C_0805_2012Metric" H 3938 2850 50  0001 C CNN
+F 2 "Capacitor_SMD:C_0402_1005Metric" H 3938 2850 50  0001 C CNN
 F 3 "" H 3900 3000 50  0001 C CNN
 	1    3900 3000
@@
 F 0 "C5" H 8350 3850 50  0000 L CNN
 F 1 "0.1uF" H 8350 3650 50  0000 L CNN
-F 2 "Capacitor_SMD:C_0805_2012Metric" H 8388 3600 50  0001 C CNN
+F 2 "Capacitor_SMD:C_0402_1005Metric" H 8388 3600 50  0001 C CNN
 F 3 "" H 8350 3750 50  0001 C CNN
 	1    8350 3750
@@
 F 0 "C6" H 8600 3850 50  0000 L CNN
 F 1 "0.1uF" H 8600 3650 50  0000 L CNN
-F 2 "Capacitor_SMD:C_0805_2012Metric" H 8638 3600 50  0001 C CNN
+F 2 "Capacitor_SMD:C_0402_1005Metric" H 8638 3600 50  0001 C CNN
 F 3 "" H 8600 3750 50  0001 C CNN
 	1    8600 3750
@@
 F 0 "C7" H 8850 3850 50  0000 L CNN
 F 1 "0.1uF" H 8850 3650 50  0000 L CNN
-F 2 "Capacitor_SMD:C_0805_2012Metric" H 8888 3600 50  0001 C CNN
+F 2 "Capacitor_SMD:C_0402_1005Metric" H 8888 3600 50  0001 C CNN
 F 3 "" H 8850 3750 50  0001 C CNN
 	1    8850 3750
@@
 F 0 "C9" H 9100 3850 50  0000 L CNN
 F 1 "0.1uF" H 9100 3650 50  0000 L CNN
-F 2 "Capacitor_SMD:C_0805_2012Metric" H 9138 3600 50  0001 C CNN
+F 2 "Capacitor_SMD:C_0402_1005Metric" H 9138 3600 50  0001 C CNN
 F 3 "" H 9100 3750 50  0001 C CNN
 	1    9100 3750
@@
 F 0 "C3" H 4200 2300 50  0000 L CNN
 F 1 "0.1uF" H 4200 2100 50  0000 L CNN
-F 2 "Capacitor_SMD:C_0805_2012Metric" H 4238 2050 50  0001 C CNN
+F 2 "Capacitor_SMD:C_0402_1005Metric" H 4238 2050 50  0001 C CNN
 F 3 "" H 4200 2200 50  0001 C CNN
 	1    4200 2200
@@
 F 0 "C8" H 9000 2800 50  0000 L CNN
 F 1 "0.1uF" H 9000 2600 50  0000 L CNN
-F 2 "Capacitor_SMD:C_0805_2012Metric" H 9038 2550 50  0001 C CNN
+F 2 "Capacitor_SMD:C_0402_1005Metric" H 9038 2550 50  0001 C CNN
 F 3 "" H 9000 2700 50  0001 C CNN
 	1    9000 2700

Commit message: loger desc, new pcb for remote
Parts:
- J2: footprint Connector_PinHeader_2.54mm:PinHeader_1x03_P2.54mm_Horizontal -> Connector_PinHeader_2.54mm:PinHeader_1x03_P2.54mm_Vertical
Changed lines of the file:
@@
 F 0 "J2" H 7380 5142 50  0000 L CNN
 F 1 "power_sw" H 7380 5051 50  0000 L CNN
-F 2 "Connector_PinHeader_2.54mm:PinHeader_1x03_P2.54mm_Horizontal" H 7300 5100 50  0001 C CNN
+F 2 "Connector_PinHeader_2.54mm:PinHeader_1x03_P2.54mm_Vertical" H 7300 5100 50  0001 C CNN
 F 3 "~" H 7300 5100 50  0001 C CNN
 	1    7300 5100

Commit message: two layer IR, USB CDC almost compl
Connections:
- net GND: now also U1.41 (PB5); no longer U1.12 (PA2)
- net PWR: now also U1.42 (PB6); no longer U1.46 (PB9)
- net SWDIO: no longer U1.45 (PB8)
Changed lines of the file:
@@
 NoConn ~ 4450 3800
 NoConn ~ 4450 3900
-NoConn ~ 4450 4000
-NoConn ~ 4450 4100
-Entry Wire Line
-	4100 4500 4200 4400
 Entry Wire Line
 	5800 3700 5900 3800
@@
 DP
 NoConn ~ 4450 5000
-Text Label 4250 4400 0    50   ~ 0
+Text Label 4200 4100 0    50   ~ 0
 PWR
 Wire Wire Line
@@
 Text Label 6400 5450 0    50   ~ 0
 PWR
-Text Label 4200 4300 0    50   ~ 0
-SWDIO
-Wire Wire Line
-	4450 4300 4200 4300
 $Comp
 L local:STM32F103C8Tx_usb U1
@@
 $EndComp
 Wire Wire Line
-	4200 4400 4450 4400
-Wire Wire Line
 	5550 3500 5800 3500
-Text Label 5600 3700 0    50   ~ 0
+Text Label 4200 4000 0    50   ~ 0
 GND
 Text Label 4200 5450 0    50   ~ 0
@@
 	5800 3500 5900 3600
 Entry Wire Line
-	4100 4400 4200 4300
-Entry Wire Line
 	5800 4500 5900 4600
 Wire Wire Line
 	5550 4500 5800 4500
+Wire Wire Line
+	4450 4100 4200 4100
+Entry Wire Line
+	4100 4200 4200 4100
+NoConn ~ 4450 4400
+NoConn ~ 4450 4300
 Wire Bus Line
 	4150 5750 6450 5750
+Entry Wire Line
+	4100 4100 4200 4000
+Wire Wire Line
+	4200 4000 4450 4000
 Wire Bus Line
-	4100 4350 4100 5700
+	4100 4050 4100 5700
 Wire Bus Line
 	6300 2900 6300 5700

Commit message: убрался в файлах
Parts:
- removed U3: TSOP17xx, OptoDevice:Vishay_CAST-3Pin, symbol Interface_Optical:TSOP17xx
- added U3: TSOP41xx, OptoDevice:Vishay_MOLD-3Pin, symbol Interface_Optical:TSOP41xx
Connections:
- net +3V3: now also U3.3 (Vs)
- net GND: now also U3.2 (GND)
- net IR: now also U3.1 (OUT)
Changed lines of the file:
@@
 	1    0    0    -1
-$EndComp
-$Comp
-L Interface_Optical:TSOP17xx U3
-U 1 1 61EC21C1
-P 7500 4450
-F 0 "U3" H 7750 4750 50  0000 C CNN
-F 1 "TSOP17xx" H 7300 4750 50  0000 C CNN
-F 2 "OptoDevice:Vishay_CAST-3Pin" H 7450 4075 50  0001 C CNN
-F 3 "http://www.micropik.com/PDF/tsop17xx.pdf" H 8150 4750 50  0001 C CNN
-	1    7500 4450
-	-1   0    0    -1
 $EndComp
 Wire Wire Line
@@
 NoConn ~ 4450 4400
 NoConn ~ 4450 4300
+Entry Wire Line
+	4100 4100 4200 4000
+Wire Wire Line
+	4200 4000 4450 4000
 Wire Bus Line
 	4150 5750 6450 5750
-Entry Wire Line
-	4100 4100 4200 4000
-Wire Wire Line
-	4200 4000 4450 4000
+$Comp
+L Interface_Optical:TSOP41xx U3
+U 1 1 625F74B2
+P 7500 4450
+F 0 "U3" H 7034 4500 50  0000 R CNN
+F 1 "TSOP41xx" H 7034 4409 50  0000 R CNN
+F 2 "OptoDevice:Vishay_MOLD-3Pin" H 7450 4075 50  0001 C CNN
+F 3 "http://www.vishay.com/docs/82460/tsop45.pdf" H 8150 4750 50  0001 C CNN
+	1    7500 4450
+	-1   0    0    -1
+$EndComp
 Wire Bus Line
 	4100 4050 4100 5700
