File: sch/ambilight/ambilight.kicad_pcb (KiCad board)
At the start: 2 copper layers, 47 parts, among them J1 Conn_Coaxial_Power, J2 USB_A, J3 OV2640, J4 WS_DO, J5 WS_POWER, J6 led1, J7 led2, J8 SWD, SW1 SW_CAM, SW5 SW_ON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

Commit message: ambilight buttons
Parts:
- added SW2: SW_R, local:smd_sw_ali, F.Cu at (107.2, 84.1)
- added SW3: SW_G, local:smd_sw_ali, F.Cu at (115.7, 84.1)
- added SW4: SW_B, local:smd_sw_ali, F.Cu at (124.3, 84.1)
- SW1, SW5: footprint Button_Switch_SMD:Panasonic_EVQPUJ_EVQPUA -> local:smd_sw_ali
- moved C11 2.24 mm to (115.4, 74.1)
- moved C4 2.24 mm to (115.1, 75.6)
- moved C7 2.24 mm to (111.7, 75.6)
- moved C8 2.24 mm to (108.4, 74.1)
- moved U1 2.24 mm to (115.1, 78.6)
- moved U3 2.24 mm to (108.1, 78.6)
- moved U4 2.24 mm to (111.6, 78.6)
- moved C6 2.24 mm to (108.1, 75.6)
- moved C2 2.22 mm to (117.9, 78.6)
- moved SW1 1.49 mm to (100.8, 48.1)
- moved SW5 1.29 mm to (101.1, 79.8)
- moved R10 0.37 mm to (127.0, 65.0)
- moved D1 0.23 mm to (100.5, 42.1)
Routing:
- net /SW_B: track 0.00 -> 46.0 mm, vias 0 -> 2
- net /SW_G: track 0.00 -> 42.5 mm, vias 0 -> 2
- net /SW_R: track 0.00 -> 35.6 mm, vias 0 -> 2
- net GND: track 333.5 -> 338.3 mm
- net /LED1_R: track 51.8 -> 56.0 mm
- net +1V2: track 22.1 -> 17.9 mm
- net /SW_ON: track 45.4 -> 42.1 mm
- net +2V8: track 44.9 -> 42.3 mm
- net +5V: track 26.1 -> 28.1 mm
- net /LED1_B: track 41.4 -> 43.2 mm
- net /LED1_G: track 47.4 -> 46.2 mm
- net /LED_LINE: track 2.52 -> 3.19 mm
- net Net-(J4-Pad1): track 15.5 -> 14.9 mm
