File: sch/ambilight/ambilight.sch (KiCad schematic (older format))
At the start: 34 parts

Commit message: add schematic of ambilight
Parts:
- added C? (x6): 10uF, symbol Device:C
- added C? (x9): 0.1uF, symbol Device:C
- added J?: Conn_Coaxial_Power, symbol Connector:Conn_Coaxial_Power
- added J?: WS_POWER, symbol Connector_Generic:Conn_01x02
- added U?: XC6206P33MR, Package_TO_SOT_SMD:SOT-23, symbol Regulator_Linear:XC6206PxxxMR
- added U?: XC6206P122MR, Package_TO_SOT_SMD:SOT-23, symbol Regulator_Linear:XC6206PxxxMR
- added U?: XC6206P282MR, Package_TO_SOT_SMD:SOT-23, symbol Regulator_Linear:XC6206PxxxMR
- added U?: LM358, symbol Amplifier_Operational:LM358
Connections:
- net +1V2: now also C?.2, C?.2, U?.2 (VO)
- net +2V8: now also C?.2, U?.2 (VO)
- net +3V3: now also C?.2, C?.2, C?.2, C?.2, C?.2, C?.2, C?.2, U?.2 (VO), U?.3 (VI), U?.3 (VI)
- net +5V: now also C?.2, C?.2, U?.8 (V+); no longer U?.9 (COM)
- net GND: now also C?.1, C?.1, C?.1, C?.1, C?.1, C?.1, C?.1, C?.1, C?.1, C?.1, C?.1, C?.1, C?.1, C?.1, C?.1, J?.2 (Ext), J?.2 (Pin_2), U?.1 (GND), U?.1 (GND), U?.1 (GND), U?.4 (V-)
- new net: C?.2, U?.3 (VI)
- new net +5VA: C?.2, C?.2, J?.1 (In), J?.1 (Pin_1), U?.9 (COM)
Other:
- moved on the sheet: C?, D?, J?, MK?, R?, SW?, U?, U?A, Y?

Commit message: ambilight pcb
Parts:
- removed C? (x3): 0.1uF, symbol Device:C
- removed C?: 10uF, symbol Device:C
- C1, C19, C2, C4, C6, C7: renamed from C?; footprint (none) -> Capacitor_SMD:C_0805_2012Metric
- C10, C11, C12, C13, C15, C16, C21, C22, C3, C5, C8, C9: renamed from C?; footprint (none) -> Capacitor_SMD:C_0402_1005Metric
- D1: renamed from D?; footprint (none) -> LED_SMD:LED_0805_2012Metric
- J1, J5: renamed from J?; footprint (none) -> Connector_PinHeader_2.54mm:PinHeader_1x02_P2.54mm_Vertical
- J2: renamed from J?; footprint (none) -> Connector_PinHeader_2.54mm:PinHeader_1x04_P2.54mm_Vertical
- J3: renamed from J?; footprint (none) -> Connector_FFC-FPC:Hirose_FH12-24S-0.5SH_1x24-1MP_P0.50mm_Horizontal
- J4: renamed from J?; footprint (none) -> Connector_PinHeader_2.54mm:PinHeader_1x01_P2.54mm_Vertical
- J6, J7: renamed from J?; footprint (none) -> Connector_PinHeader_2.54mm:PinHeader_1x03_P2.54mm_Vertical
- J8: renamed from J?; footprint (none) -> local:3WIRE_PADS
- MK1: renamed from MK?; footprint (none) -> Capacitor_THT:CP_Radial_D5.0mm_P2.50mm
- R1, R10, R2, R3, R4, R5, R6, R7, R8, R9: renamed from R?; footprint (none) -> Resistor_SMD:R_0402_1005Metric
- SW1, SW2, SW3, SW4, SW5: renamed from SW?; footprint (none) -> Button_Switch_SMD:Panasonic_EVQPUJ_EVQPUA
- U2: renamed from U?; footprint (none) -> Package_SO:SO-8_3.9x4.9mm_P1.27mm
- U6: renamed from U?; footprint (none) -> Package_SO:SOIC-16_3.9x9.9mm_P1.27mm
- Y1: renamed from Y?; footprint (none) -> Crystal:Crystal_SMD_5032-2Pin_5.0x3.2mm
- gave numbers to parts that had none: 4
Connections:
- net +3V3: now also R1.2, R5.2, U2.8 (V+); no longer U3.3 (VI), U4.3 (VI)
- net +5V: now also C2.2, U1.3 (VI), U3.3 (VI), U4.3 (VI); no longer R1.2, R5.2, U2.8 (V+)
- net LED1_B: now also U6.6 (I6); no longer U6.3 (I3)
- net LED1_G: now also U6.5 (I5); no longer U6.2 (I2)
- net LED1_R: now also U6.4 (I4); no longer U6.1 (I1)
- net LED2_B: now also U6.3 (I3); no longer U6.6 (I6)
- net LED2_G: now also U6.2 (I2); no longer U6.5 (I5)
- net LED2_R: now also U6.1 (I1); no longer U6.4 (I4)
Other:
- moved on the sheet: C15, C16, C19, C2, C4, C5, C6, C7, C8, U1, U3, U4

Commit message: ambilight buttons
Parts:
- SW1, SW2, SW3, SW4, SW5: footprint Button_Switch_SMD:Panasonic_EVQPUJ_EVQPUA -> local:smd_sw_ali
Changed lines of the file:
@@
 F 0 "SW2" H 2100 2850 50  0000 C CNN
 F 1 "SW_R" H 2400 2850 50  0000 C CNN
-F 2 "Button_Switch_SMD:Panasonic_EVQPUJ_EVQPUA" H 2250 2950 50  0001 C CNN
+F 2 "local:smd_sw_ali" H 2250 2950 50  0001 C CNN
 F 3 "~" H 2250 2950 50  0001 C CNN
 	1    2250 2750
@@
 F 0 "SW3" H 2100 3050 50  0000 C CNN
 F 1 "SW_G" H 2400 3050 50  0000 C CNN
-F 2 "Button_Switch_SMD:Panasonic_EVQPUJ_EVQPUA" H 2250 3150 50  0001 C CNN
+F 2 "local:smd_sw_ali" H 2250 3150 50  0001 C CNN
 F 3 "~" H 2250 3150 50  0001 C CNN
 	1    2250 2950
@@
 F 0 "SW4" H 2100 3250 50  0000 C CNN
 F 1 "SW_B" H 2400 3250 50  0000 C CNN
-F 2 "Button_Switch_SMD:Panasonic_EVQPUJ_EVQPUA" H 2250 3350 50  0001 C CNN
+F 2 "local:smd_sw_ali" H 2250 3350 50  0001 C CNN
 F 3 "~" H 2250 3350 50  0001 C CNN
 	1    2250 3150
@@
 F 0 "SW5" H 2100 3450 50  0000 C CNN
 F 1 "SW_ON" H 2500 3450 50  0000 C CNN
-F 2 "Button_Switch_SMD:Panasonic_EVQPUJ_EVQPUA" H 2250 3550 50  0001 C CNN
+F 2 "local:smd_sw_ali" H 2250 3550 50  0001 C CNN
 F 3 "~" H 2250 3550 50  0001 C CNN
 	1    2250 3350
@@
 F 0 "SW1" H 2100 2650 50  0000 C CNN
 F 1 "SW_CAM" H 2500 2650 50  0000 C CNN
-F 2 "Button_Switch_SMD:Panasonic_EVQPUJ_EVQPUA" H 2250 2750 50  0001 C CNN
+F 2 "local:smd_sw_ali" H 2250 2750 50  0001 C CNN
 F 3 "~" H 2250 2750 50  0001 C CNN
 	1    2250 2550
